Commit message: reduced limits

File: robots/iiwa.urdf (robot description, URDF)
Before this commit: robot iiwa14, 10 links, 9 joints
Joints:
- joint iiwa_joint_1: limit lower=-2.9670597283903604 upper=2.9670597283903604 effort=300 velocity=10 -> lower=-2.9321531433504737 upper=2.9321531433504737 effort=300 velocity=10
- joint iiwa_joint_2: limit lower=-2.0943951023931953 upper=2.0943951023931953 effort=300 velocity=10 -> lower=-2.0594885173533086 upper=2.0594885173533086 effort=300 velocity=10
- joint iiwa_joint_3: limit lower=-2.9670597283903604 upper=2.9670597283903604 effort=300 velocity=10 -> lower=-2.9321531433504737 upper=2.9321531433504737 effort=300 velocity=10
- joint iiwa_joint_4: limit lower=-2.0943951023931953 upper=2.0943951023931953 effort=300 velocity=10 -> lower=-2.0594885173533086 upper=2.0594885173533086 effort=300 velocity=10
- joint iiwa_joint_5: limit lower=-2.9670597283903604 upper=2.9670597283903604 effort=300 velocity=10 -> lower=-2.9321531433504737 upper=2.9321531433504737 effort=300 velocity=10
- joint iiwa_joint_6: limit lower=-2.0943951023931953 upper=2.0943951023931953 effort=300 velocity=10 -> lower=-2.0594885173533086 upper=2.0594885173533086 effort=300 velocity=10
- joint iiwa_joint_7: limit lower=-3.0543261909900763 upper=3.0543261909900763 effort=300 velocity=10 -> lower=-3.01941960595019 upper=3.01941960595019 effort=300 velocity=10
